Commit message: add HDR10L-19, HDR20-17 models

File: urdf/robots/ha006b/ha006b.urdf.xacro (robot description, xacro)
@@ -1,6 +1,6 @@
 <?xml version='1.0' encoding='utf-8'?>
 <robot name="hdr_robot" xmlns:xacro="http://ros.org/wiki/xacro">
-  <material name="white">
-    <color rgba="1.0 1.0 1.0 1.0" />
+  <material name="ivory">
+    <color rgba="1.0 0.945 0.773 1.0" />
   </material>
   <material name="black">
@@ -16,5 +16,5 @@
         <mesh filename="file://$(find hdr_description)/meshes/robots/ha006b/visual/base_body.stl" scale="${mesh_scale} ${mesh_scale} ${mesh_scale}" />
       </geometry>
-      <material name="white" />
+      <material name="ivory" />
     </visual>
     <collision>
@@ -34,5 +34,5 @@
         <mesh filename="file://$(find hdr_description)/meshes/robots/ha006b/visual/lower_frame.stl" scale="${mesh_scale} ${mesh_scale} ${mesh_scale}" />
       </geometry>
-      <material name="white" />
+      <material name="ivory" />
     </visual>
     <collision>
@@ -52,5 +52,5 @@
         <mesh filename="file://$(find hdr_description)/meshes/robots/ha006b/visual/upper_frame.stl" scale="${mesh_scale} ${mesh_scale} ${mesh_scale}" />
       </geometry>
-      <material name="white" />
+      <material name="ivory" />
     </visual>
     <collision>
@@ -70,5 +70,5 @@
         <mesh filename="file://$(find hdr_description)/meshes/robots/ha006b/visual/arm.stl" scale="${mesh_scale} ${mesh_scale} ${mesh_scale}" />
       </geometry>
-      <material name="white" />
+      <material name="ivory" />
     </visual>
     <collision>
@@ -88,5 +88,5 @@
         <mesh filename="file://$(find hdr_description)/meshes/robots/ha006b/visual/wrist_body.stl" scale="${mesh_scale} ${mesh_scale} ${mesh_scale}" />
       </geometry>
-      <material name="white" />
+      <material name="ivory" />
     </visual>
     <collision>
@@ -106,5 +106,5 @@
         <mesh filename="file://$(find hdr_description)/meshes/robots/ha006b/visual/wrist_holder.stl" scale="${mesh_scale} ${mesh_scale} ${mesh_scale}" />
       </geometry>
-      <material name="white" />
+      <material name="ivory" />
     </visual>
     <collision>

File: urdf/robots/hdr10l_19/hdr10l_19.urdf.xacro (robot description, xacro)
@@ -4,27 +4,27 @@
     <color rgba="1.0 0.945 0.773 1.0" />
   </material>
+  <material name="black">
+    <color rgba="0.2 0.2 0.2 1.0"/>
+  </material>
   <material name="gray">
     <color rgba="0.3 0.3 0.3 1.0"/>
   </material>
-  <material name="black">
-    <color rgba="0.2 0.2 0.2 1.0"/>
-  </material>
   <xacro:property name="mesh_scale" value="0.001" />
   <link name="base_link">
     <visual>
       <geometry>
-        <mesh filename="file://$(find hdr_description)/meshes/robots/hh020/visual/base_body.stl" scale="${mesh_scale} ${mesh_scale} ${mesh_scale}"/>
-      </geometry>
-      <material name="ivory"/>
-    </visual>
-    <collision>
-      <geometry>
-        <mesh filename="file://$(find hdr_description)/meshes/robots/hh020/collision/base_body.stl" scale="${mesh_scale} ${mesh_scale} ${mesh_scale}"/>
-      </geometry>
-    </collision>
-    <inertial>
-      <mass value="31.2543"/>
-      <origin xyz="0 0 0" rpy="0 0 0"/>
-      <inertia ixx="0.4278" ixy="0" ixz="0" iyy="0.7085" iyz="0" izz="0.8249"/>
+        <mesh filename="file://$(find hdr_description)/meshes/robots/hdr10l_19/visual/base_body.stl" scale="${mesh_scale} ${mesh_scale} ${mesh_scale}"/>
+      </geometry>
+      <material name="ivory"/>
+    </visual>
+    <collision>
+      <geometry>
+        <mesh filename="file://$(find hdr_description)/meshes/robots/hdr10l_19/collision/base_body.stl" scale="${mesh_scale} ${mesh_scale} ${mesh_scale}"/>
+      </geometry>
+    </collision>
+    <inertial>
+      <mass value="44.0197"/>
+      <origin xyz="0 0 0" rpy="0 0 0"/>
+      <inertia ixx="0.5025" ixy="0" ixz="0" iyy="0.8947" iyz="0" izz="1.1434"/>
     </inertial>
   </link>
@@ -32,11 +32,11 @@
     <visual>
       <geometry>
-        <mesh filename="file://$(find hdr_description)/meshes/robots/hh020/visual/lower_frame.stl" scale="${mesh_scale} ${mesh_scale} ${mesh_scale}"/>
-      </geometry>
-      <material name="ivory"/>
-    </visual>
-    <collision>
-      <geometry>
-        <mesh filename="file://$(find hdr_description)/meshes/robots/hh020/collision/lower_frame.stl" scale="${mesh_scale} ${mesh_scale} ${mesh_scale}"/>
+        <mesh filename="file://$(find hdr_description)/meshes/robots/hdr10l_19/visual/lower_frame.stl" scale="${mesh_scale} ${mesh_scale} ${mesh_scale}"/>
+      </geometry>
+      <material name="ivory"/>
+    </visual>
+    <collision>
+      <geometry>
+        <mesh filename="file://$(find hdr_description)/meshes/robots/hdr10l_19/collision/lower_frame.stl" scale="${mesh_scale} ${mesh_scale} ${mesh_scale}"/>
       </geometry>
     </collision>
@@ -44,17 +44,19 @@
       <mass value="44.2299"/>
       <origin xyz="0 0 0" rpy="0 0 0"/>
-      <inertia ixx="1.046" ixy="0" ixz="0" iyy="1.046" iyz="0" izz="1.1643"/>
+      <inertia ixx="1.0415" ixy="0" ixz="0" iyy="1.3015" iyz="0" izz="1.163"/>
     </inertial>
   </link>
   <link name="upper_frame_link">
     <visual>
-      <geometry>
-        <mesh filename="file://$(find hdr_description)/meshes/robots/hh020/visual/upper_frame.stl" scale="${mesh_scale} ${mesh_scale} ${mesh_scale}"/>
-      </geometry>
-      <material name="ivory"/>
-    </visual>
-    <collision>
-      <geometry>
-        <mesh filename="file://$(find hdr_description)/meshes/robots/hh020/collision/upper_frame.stl" scale="${mesh_scale} ${mesh_scale} ${mesh_scale}"/>
+      <origin xyz="-0.16 0 -0.4466" rpy="0 0 0"/>
+      <geometry>
+        <mesh filename="file://$(find hdr_description)/meshes/robots/hdr10l_19/visual/upper_frame.stl" scale="${mesh_scale} ${mesh_scale} ${mesh_scale}"/>
+      </geometry>
+      <material name="ivory"/>
+    </visual>
+    <collision>
+      <origin xyz="-0.16 0 -0.4466" rpy="0 0 0"/>
+      <geometry>
+        <mesh filename="file://$(find hdr_description)/meshes/robots/hdr10l_19/collision/upper_frame.stl" scale="${mesh_scale} ${mesh_scale} ${mesh_scale}"/>
       </geometry>
     </collision>
@@ -62,17 +64,19 @@
       <mass value="22.4028"/>
       <origin xyz="0 0 0" rpy="0 0 0"/>
-      <inertia ixx="1.8777" ixy="0" ixz="0" iyy="1.9502" iyz="0" izz="0.1647"/>
+      <inertia ixx="1.8615" ixy="0" ixz="0" iyy="1.9502" iyz="0" izz="0.1485"/>
     </inertial>
   </link>
   <link name="arm_link">
     <visual>
-      <geometry>
-        <mesh filename="file://$(find hdr_description)/meshes/robots/hh020/visual/arm.stl" scale="${mesh_scale} ${mesh_scale} ${mesh_scale}"/>
-      </geometry>
-      <material name="ivory"/>
-    </visual>
-    <collision>
-      <geometry>
-        <mesh filename="file://$(find hdr_description)/meshes/robots/hh020/collision/arm.stl" scale="${mesh_scale} ${mesh_scale} ${mesh_scale}"/>
+      <origin xyz="-0.16 0 -1.217" rpy="0 0 0"/>
+      <geometry>
+        <mesh filename="file://$(find hdr_description)/meshes/robots/hdr10l_19/visual/arm.stl" scale="${mesh_scale} ${mesh_scale} ${mesh_scale}"/>
+      </geometry>
+      <material name="ivory"/>
+    </visual>
+    <collision>
+      <origin xyz="-0.16 0 -1.216" rpy="0 0 0"/>
+      <geometry>
+        <mesh filename="file://$(find hdr_description)/meshes/robots/hdr10l_19/collision/arm.stl" scale="${mesh_scale} ${mesh_scale} ${mesh_scale}"/>
       </geometry>
     </collision>
@@ -80,19 +84,19 @@
       <mass value="14.2656"/>
       <origin xyz="0 0 0" rpy="0 0 0"/>
-      <inertia ixx="0.1905" ixy="0" ixz="0" iyy="0.2375" iyz="0" izz="0.1845"/>
+      <inertia ixx="0.1949" ixy="0" ixz="0" iyy="0.239" iyz="0" izz="0.1873"/>
     </inertial>
   </link>
   <link name="wrist_body_link">
     <visual>
-      <origin xyz="-0.162 0 0" rpy="0 0 0"/>
-      <geometry>
-        <mesh filename="file://$(find hdr_description)/meshes/robots/hh020/visual/wrist_body.stl" scale="${mesh_scale} ${mesh_scale} ${mesh_scale}"/>
-      </geometry>
-      <material name="ivory"/>
-    </visual>
-    <collision>
-      <origin xyz="-0.162 0 0" rpy="0 0 0"/>
-      <geometry>
-        <mesh filename="file://$(find hdr_description)/meshes/robots/hh020/collision/wrist_body.stl" scale="${mesh_scale} ${mesh_scale} ${mesh_scale}"/>
+      <origin xyz="-0.162 0 -1.3565" rpy="0 0 0"/>
+      <geometry>
+        <mesh filename="file://$(find hdr_description)/meshes/robots/hdr10l_19/visual/wrist_body.stl" scale="${mesh_scale} ${mesh_scale} ${mesh_scale}"/>
+      </geometry>
+      <material name="ivory"/>
+    </visual>
+    <collision>
+      <origin xyz="-0.142 0 -1.3565" rpy="0 0 0"/>
+      <geometry>
+        <mesh filename="file://$(find hdr_description)/meshes/robots/hdr10l_19/collision/wrist_body.stl" scale="${mesh_scale} ${mesh_scale} ${mesh_scale}"/>
       </geometry>
     </collision>
@@ -100,19 +104,19 @@
       <mass value="7.0632"/>
       <origin xyz="0 0 0" rpy="0 0 0"/>
-      <inertia ixx="0.0347" ixy="0" ixz="0" iyy="0.2705" iyz="0" izz="0.281"/>
+      <inertia ixx="0.0244" ixy="0" ixz="0" iyy="0.49" iyz="0" izz="0.49"/>
     </inertial>
   </link>
   <link name="wrist_holder_link">
     <visual>
-      <origin xyz="0.00186 0 0.0022" rpy="0 0 0"/>
-      <geometry>
-        <mesh filename="file://$(find hdr_description)/meshes/robots/hh020/visual/wrist_holder.stl" scale="${mesh_scale} ${mesh_scale} ${mesh_scale}"/>
-      </geometry>
-      <material name="ivory"/>
-    </visual>
-    <collision>
-      <origin xyz="0.00186 0 0.0022" rpy="0 0 0"/>
-      <geometry>
-        <mesh filename="file://$(find hdr_description)/meshes/robots/hh020/collision/wrist_holder.stl" scale="${mesh_scale} ${mesh_scale} ${mesh_scale}"/>
+      <origin xyz="-1.215 0 -1.356" rpy="0 0 0"/>
+      <geometry>
+        <mesh filename="file://$(find hdr_description)/meshes/robots/hdr10l_19/visual/wrist_holder.stl" scale="${mesh_scale} ${mesh_scale} ${mesh_scale}"/>
+      </geometry>
+      <material name="ivory"/>
+    </visual>
+    <collision>
+      <origin xyz="-1.215 0 -1.356" rpy="0 0 0"/>
+      <geometry>
+        <mesh filename="file://$(find hdr_description)/meshes/robots/hdr10l_19/collision/wrist_holder.stl" scale="${mesh_scale} ${mesh_scale} ${mesh_scale}"/>
       </geometry>
     </collision>
@@ -120,17 +124,19 @@
       <mass value="3.8171"/>
       <origin xyz="0 0 0" rpy="0 0 0"/>
-      <inertia ixx="0.0087" ixy="0" ixz="0" iyy="0.0172" iyz="0" izz="0.0182"/>
+      <inertia ixx="0.0046" ixy="0" ixz="0" iyy="0.0097" iyz="0" izz="0.0087"/>
     </inertial>
   </link>
   <link name="flange_link">
     <visual>
-      <geometry>
-        <mesh filename="file://$(find hdr_description)/meshes/robots/hh020/visual/flange.stl" scale="${mesh_scale} ${mesh_scale} ${mesh_scale}"/>
+      <origin xyz="-1.318 0 -1.356" rpy="0 0 0"/>
+      <geometry>
+        <mesh filename="file://$(find hdr_description)/meshes/robots/hdr10l_19/visual/flange.stl" scale="${mesh_scale} ${mesh_scale} ${mesh_scale}"/>
       </geometry>
       <material name="gray"/>
     </visual>
     <collision>
-      <geometry>
-        <mesh filename="file://$(find hdr_description)/meshes/robots/hh020/collision/flange.stl" scale="${mesh_scale} ${mesh_scale} ${mesh_scale}"/>
+      <origin xyz="-1.318 0 -1.356" rpy="0 0 0"/>
+      <geometry>
+        <mesh filename="file://$(find hdr_description)/meshes/robots/hdr10l_19/collision/flange.stl" scale="${mesh_scale} ${mesh_scale} ${mesh_scale}"/>
       </geometry>
     </collision>
@@ -138,5 +144,5 @@
       <mass value="0.4672"/>
       <origin xyz="0 0 0" rpy="0 0 0"/>
-      <inertia ixx="0.0002" ixy="0" ixz="0" iyy="0.0001" iyz="0" izz="0.0001"/>
+      <inertia ixx="0.0002" ixy="0" ixz="0" iyy="0.0002" iyz="0" izz="0.0002"/>
     </inertial>
   </link>
@@ -144,5 +150,5 @@
     <visual>
       <geometry>
-        <mesh filename="file://$(find hdr_description)/meshes/robots/hh020/visual/motor_s.stl" scale="${mesh_scale} ${mesh_scale} ${mesh_scale}"/>
+        <mesh filename="file://$(find hdr_description)/meshes/robots/hdr10l_19/visual/motor_s.stl" scale="${mesh_scale} ${mesh_scale} ${mesh_scale}"/>
       </geometry>
       <material name="black"/>
@@ -150,5 +156,5 @@
     <collision>
       <geometry>
-        <mesh filename="file://$(find hdr_description)/meshes/robots/hh020/collision/motor_s.stl" scale="${mesh_scale} ${mesh_scale} ${mesh_scale}"/>
+        <mesh filename="file://$(find hdr_description)/meshes/robots/hdr10l_19/collision/motor_s.stl" scale="${mesh_scale} ${mesh_scale} ${mesh_scale}"/>
       </geometry>
     </collision>
@@ -162,5 +168,5 @@
     <visual>
       <geometry>
-        <mesh filename="file://$(find hdr_description)/meshes/robots/hh020/visual/motor_h.stl" scale="${mesh_scale} ${mesh_scale} ${mesh_scale}"/>
+        <mesh filename="file://$(find hdr_description)/meshes/robots/hdr10l_19/visual/motor_h.stl" scale="${mesh_scale} ${mesh_scale} ${mesh_scale}"/>
       </geometry>
       <material name="black"/>
@@ -168,5 +174,5 @@
     <collision>
       <geometry>
-        <mesh filename="file://$(find hdr_description)/meshes/robots/hh020/collision/motor_h.stl" scale="${mesh_scale} ${mesh_scale} ${mesh_scale}"/>
+        <mesh filename="file://$(find hdr_description)/meshes/robots/hdr10l_19/collision/motor_h.stl" scale="${mesh_scale} ${mesh_scale} ${mesh_scale}"/>
       </geometry>
     </collision>
@@ -179,12 +185,14 @@
   <link name="motor_v">
     <visual>
-      <geometry>
-        <mesh filename="file://$(find hdr_description)/meshes/robots/hh020/visual/motor_v.stl" scale="${mesh_scale} ${mesh_scale} ${mesh_scale}"/>
+      <origin xyz="-0.16 0 -1.21" rpy="0 0 0"/>
+      <geometry>
+        <mesh filename="file://$(find hdr_description)/meshes/robots/hdr10l_19/visual/motor_v.stl" scale="${mesh_scale} ${mesh_scale} ${mesh_scale}"/>
       </geometry>
       <material name="black"/>
     </visual>
     <collision>
-      <geometry>
-        <mesh filename="file://$(find hdr_description)/meshes/robots/hh020/collision/motor_v.stl" scale="${mesh_scale} ${mesh_scale} ${mesh_scale}"/>
+      <origin xyz="-0.16 0 -1.21" rpy="0 0 0"/>
+      <geometry>
+        <mesh filename="file://$(find hdr_description)/meshes/robots/hdr10l_19/collision/motor_v.stl" scale="${mesh_scale} ${mesh_scale} ${mesh_scale}"/>
       </geometry>
     </collision>
@@ -200,40 +208,40 @@
     <origin xyz="0 0 0" rpy="0 0 0"/>
     <axis xyz="0 0 1"/>
-    <limit lower="-3.229" upper="3.229" effort="962.91" velocity="3.316"/>
+    <limit lower="-3.228" upper="3.228" effort="962.8" velocity="3.665"/>
   </joint>
   <joint name="j2" type="revolute">
     <parent link="lower_frame_link"/>
     <child link="upper_frame_link"/>
-    <origin xyz="0.160 0 0.4466" rpy="0 1.5708 0"/>
+    <origin xyz="0.16 0 0.4466" rpy="0 1.5708 0"/>
     <axis xyz="0 -1 0"/>
-    <limit lower="-1.222" upper="3.403" effort="1043.28" velocity="3.142"/>
+    <limit lower="-1.221" upper="3.403" effort="1010.9" velocity="3.665"/>
   </joint>
   <joint name="j3" type="revolute">
     <parent link="upper_frame_link"/>
     <child link="arm_link"/>
-    <origin xyz="0 0 0.770" rpy="0 0 0"/>
+    <origin xyz="0 0 0.77" rpy="0 0 0"/>
     <axis xyz="0 -1 0"/>
-    <limit lower="-1.396" upper="3.141" effort="538.056" velocity="3.316"/>
+    <limit lower="-1.396" upper="3.142" effort="934.1" velocity="3.84"/>
   </joint>
   <joint name="j4" type="revolute">
     <parent link="arm_link"/>
     <child link="wrist_body_link"/>
-    <origin xyz="0 0 0.140" rpy="0 0 0"/>
-    <axis xyz="1 0 0"/>
-    <limit lower="-3.403" upper="3.403" effort="44.91" velocity="6.632"/>
+    <origin xyz="0 0 0.14" rpy="0 0 0"/>
+    <axis xyz="1 0 0"/>
+    <limit lower="-3.403" upper="3.403" effort="91.3" velocity="7.33"/>
   </joint>
   <joint name="j5" type="revolute">
     <parent link="wrist_body_link"/>
     <child link="wrist_holder_link"/>
-    <origin xyz="0.8 0 0" rpy="0 0 0"/>
+    <origin xyz="1.055 0 0" rpy="0 0 0"/>
     <axis xyz="0 -1 0"/>
-    <limit lower="-2.356" upper="2.356" effort="43.52" velocity="6.632"/>
+    <limit lower="-2.356" upper="2.356" effort="20.6" velocity="7.854"/>
   </joint>
   <joint name="j6" type="revolute">
     <parent link="wrist_holder_link"/>
     <child link="flange_link"/>
-    <origin xyz="0.112 0 0" rpy="0 0 0"/>
-    <axis xyz="1 0 0"/>
-    <limit lower="-6.283" upper="6.283" effort="25.6" velocity="10.472"/>
+    <origin xyz="0.105 0 0" rpy="0 0 0"/>
+    <axis xyz="1 0 0"/>
+    <limit lower="-6.283" upper="6.283" effort="10.0" velocity="12.566"/>
   </joint>
   <joint name="joint_motor_s" type="fixed">
@@ -250,7 +258,7 @@
   </joint>
   <joint name="joint_motor_v" type="fixed">
-    <parent link="upper_frame_link"/>
+    <parent link="arm_link"/>
     <child link="motor_v"/>
-    <origin xyz="-0.16 0 -0.4466" rpy="0 0 0"/>
+    <origin xyz="0 0 0" rpy="0 0 0"/>
     <axis xyz="1 0 0"/>
   </joint>
